Commit message: prepare experiment on real robot

File: 03-control_under_collisions/panda_arm_hand.urdf (robot description, URDF)
Before this commit: robot panda_hand, 10 links, 9 joints
Links:
- link link2: geometry collision mesh filename=../../../Model/meshes/link2.obj; visual mesh filename=../../../Model/meshes/link2.obj
- link link5: geometry collision mesh filename=../../../Model/meshes/link5.obj; visual mesh filename=../../../Model/meshes/link5.obj
