Commit message: reworked applications and made compatible with latest sai2

File: 03-open_loop_force_control/panda_arm_hand.urdf (robot description, URDF)
Before this commit: robot panda_hand, 10 links, 9 joints
Links:
- link leftfinger: geometry collision mesh filename=../../../Model/meshes/collision/finger.obj; visual mesh filename=../../../Model/meshes/visual/finger.obj
- link rightfinger: geometry collision mesh filename=../../../Model/meshes/collision/finger.obj; visual mesh filename=../../../Model/meshes/visual/finger.obj

File: 06-pick_and_place/panda_arm_hand.urdf (robot description, URDF)
Before this commit: robot panda_hand, 10 links, 9 joints
Links:
- link leftfinger: geometry collision mesh filename=../../../Model/meshes/collision/finger.obj; visual mesh filename=../../../Model/meshes/visual/finger.obj
- link link0: geometry visual mesh filename=../../../Model/meshes/visual/link0.obj
- link link1: geometry visual mesh filename=../../../Model/meshes/visual/link1.obj
- link link2: geometry visual mesh filename=../../../Model/meshes/visual/link2.obj
- link link3: geometry visual mesh filename=../../../Model/meshes/visual/link3.obj
- link link4: geometry collision mesh filename=../../../Model/meshes/collision/link4.obj; visual mesh filename=../../../Model/meshes/visual/link4.obj
- link link5: geometry visual mesh filename=../../../Model/meshes/visual/link5.obj
- link link6: geometry visual mesh filename=../../../Model/meshes/visual/link6.obj
- link link7: geometry visual mesh filename=../../../Model/meshes/visual/hand.obj; visual mesh filename=../../../Model/meshes/visual/link7.obj
- link rightfinger: geometry collision mesh filename=../../../Model/meshes/collision/finger.obj; visual mesh filename=../../../Model/meshes/visual/finger.obj
Joints:
- joint finger_joint2: mimic joint=finger_joint1 -> (none)

File: 07-dual_arm_tray/panda_arm.urdf (robot description, URDF)
Before this commit: robot panda, 8 links, 7 joints
Links:
- link link0: geometry visual mesh filename=../../../Model/meshes/visual/link0.obj
- link link1: geometry visual mesh filename=../../../Model/meshes/visual/link1.obj
- link link2: geometry visual mesh filename=../../../Model/meshes/visual/link2.obj
- link link3: geometry visual mesh filename=../../../Model/meshes/visual/link3.obj
- link link4: geometry visual mesh filename=../../../Model/meshes/visual/link4.obj
- link link5: geometry visual mesh filename=../../../Model/meshes/visual/link5.obj
- link link6: geometry visual mesh filename=../../../Model/meshes/visual/link6.obj
- link link7: mass 0.5 -> 1.8; geometry visual mesh filename=../../../Model/meshes/visual/link7.obj
