Commit message: temporary electric cable simulation

File: 08-simulation_electric_cables/two_arm_panda_gripper.urdf (robot description, URDF)
Before this commit: robot two_arm_panda_gripper, 20 links, 19 joints
Links:
- link chest: geometry visual box size=0.3 0.3 1.2; visual mesh filename=../../../Model/meshes/visual/link0.obj
- link left_arm_leftfinger: geometry collision mesh filename=../../../Model/meshes/collision/finger.obj; visual mesh filename=../../../Model/meshes/collision/finger.obj
- link left_arm_rightfinger: geometry collision mesh filename=../../../Model/meshes/collision/finger.obj; visual mesh filename=../../../Model/meshes/collision/finger.obj
- link right_arm_leftfinger: geometry collision mesh filename=../../../Model/meshes/collision/finger.obj; visual mesh filename=../../../Model/meshes/collision/finger.obj
- link right_arm_rightfinger: geometry collision mesh filename=../../../Model/meshes/collision/finger.obj; visual mesh filename=../../../Model/meshes/collision/finger.obj
