Commit message: prepared tests for panda opspace

File: 02-cartesian_motion/panda_arm.urdf (robot description, URDF)
Before this commit: robot panda_hand, 10 links, 9 joints
Links:
- removed link leftfinger
- removed link rightfinger
- link link0: geometry visual mesh filename=../../../Model/meshes/visual/link0.obj
- link link1: geometry visual mesh filename=../../../Model/meshes/visual/link1.obj
- link link2: geometry visual mesh filename=../../../Model/meshes/visual/link2.obj
- link link3: geometry visual mesh filename=../../../Model/meshes/visual/link3.obj
- link link4: geometry visual mesh filename=../../../Model/meshes/visual/link4.obj
- link link5: geometry visual mesh filename=../../../Model/meshes/visual/link5.obj
- link link6: geometry visual mesh filename=../../../Model/meshes/visual/link6.obj
- link link7: mass 1.8 -> 0.5; geometry visual mesh filename=../../../Model/meshes/visual/link7.obj
Joints:
- removed joint finger_joint1
- removed joint finger_joint2

File: 02-cartesian_motion/panda_arm_hand.urdf (robot description, URDF)
Before this commit: robot panda, 8 links, 7 joints
Links:
- added link leftfinger, mass 0.1; collision mesh filename=../../../Model/meshes/collision/finger.obj; visual mesh filename=../../../Model/meshes/visual/finger.obj
- added link rightfinger, mass 0.1; collision mesh filename=../../../Model/meshes/collision/finger.obj; visual mesh filename=../../../Model/meshes/visual/finger.obj
- link link0: geometry visual mesh filename=../../../Model/meshes/visual/link0.obj
- link link1: geometry visual mesh filename=../../../Model/meshes/visual/link1.obj
- link link2: geometry visual mesh filename=../../../Model/meshes/visual/link2.obj
- link link3: geometry visual mesh filename=../../../Model/meshes/visual/link3.obj
- link link4: geometry collision mesh filename=../../../Model/meshes/collision/link4.obj; visual mesh filename=../../../Model/meshes/visual/link4.obj
- link link5: geometry visual mesh filename=../../../Model/meshes/visual/link5.obj
- link link6: geometry visual mesh filename=../../../Model/meshes/visual/link6.obj
- link link7: mass 0.5 -> 1.8; geometry visual mesh filename=../../../Model/meshes/visual/hand.obj; visual mesh filename=../../../Model/meshes/visual/link7.obj
Joints:
- added joint finger_joint1: type prismatic, parent link7, child leftfinger, origin xyz=0 0 0.1654 rpy=0 0 -0.78539816339, axis 0 1 0, limit lower=0.0 upper=0.04 effort=20 velocity=0.2
- added joint finger_joint2: type prismatic, parent link7, child rightfinger, origin xyz=0 0 0.1654 rpy=0 0 -0.78539816339, axis 0 1 0, limit lower=0.0 upper=0.04 effort=20 velocity=0.2, mimic joint=finger_joint1
