Commit message: haptic painting tested in simulation

File: 09-haptic_painting/panda_arm_brush.urdf (robot description, URDF)
Before this commit: robot panda, 8 links, 7 joints
Links:
- link link7: geometry collision cylinder length=0.4 radius=0.005; visual cylinder length=0.4 radius=0.005

File: 09-haptic_painting/panda_arm_palette.urdf (robot description, URDF)
Before this commit: robot panda, 8 links, 7 joints
Links:
- link link7: geometry collision box size=0.3 0.2 0.005; visual box size=0.3 0.2 0.005
