Commit message: finished experiments on unigrasp allegro

File: 12-uniGrasp_allegro/floatingAllegroHand.urdf (robot description, URDF)
Before this commit: robot AllegroHand, 28 links, 27 joints
Joints:
- joint virtual_ry: child virtual_link_4 -> virtual_link_6; parent virtual_link_3 -> virtual_link_5
- joint virtual_rz: child virtual_link_6 -> virtual_link_4; parent virtual_link_5 -> virtual_link_3
