Commit message: a bunch of aux applications and tests

File: 00-contact_force_estimator/panda_arm.urdf (robot description, URDF)
Before this commit: robot panda, 8 links, 7 joints
Links:
- link link7: geometry visual mesh filename=../../../Model/meshes/visual/link7.obj; visual sphere radius=0.04

File: 18-haptic_local_force_loop/panda_arm.urdf (robot description, URDF)
Before this commit: robot panda, 8 links, 7 joints
Links:
- added link end_effector, mass 0.5; collision sphere radius=0.035; visual sphere radius=0.035
- link link7: geometry visual mesh filename=../../../Model/meshes/visual/link7.obj
Joints:
- added joint joint_fixed: type fixed, parent link7, child end_effector, origin xyz=0 0 0.13 rpy=0 0 0

File: zz-two_arm_coordination_tests/panda_arm.urdf (robot description, URDF)
Before this commit: robot panda, 8 links, 7 joints
Links:
- link link7: geometry visual mesh filename=../../../Model/meshes/visual/link7.obj

File: zz-two_arm_coordination_tests/panda_arm_flat_ee.urdf (robot description, URDF)
Before this commit: robot panda, 8 links, 7 joints
Links:
- link link7: geometry collision box size=0.09 0.09 0.02; visual box size=0.09 0.09 0.02
