Commit message: prepared local-aut haptic experiments

File: 19-bracing_one_arm/panda_arm.urdf (robot description, URDF)
Before this commit: robot panda, 9 links, 8 joints
Links:
- removed link end_effector
- added link end-effector, mass 0.2; collision sphere radius=0.04; visual sphere radius=0.04
- link link4: geometry collision sphere radius=0.05; visual mesh filename=../../../Model/meshes/visual/link4.obj
Joints:
- removed joint joint_fixed
- added joint joint_ee: type fixed, parent link7, child end-effector, origin xyz=0 0 0.15 rpy=0 0 0
- joint joint1: origin xyz=0 0 0.333 rpy=0 0 0 -> xyz=0.333 0 0.8 rpy=1.57079632679 0 1.57079632679

File: 20-bracing_one_arm_floating_base/panda_arm.urdf (robot description, URDF)
Before this commit: robot panda, 9 links, 8 joints
Links:
- removed link end_effector
- added link base_link, mass 0.1
- added link end-effector, mass 0.2; collision sphere radius=0.04; visual sphere radius=0.04
- link link4: geometry collision sphere radius=0.05; visual mesh filename=../../../Model/meshes/visual/link4.obj
Joints:
- removed joint joint_fixed
- added joint base_joint: type prismatic, parent base_link, child link0, origin xyz=0.0 0.0 0.8 rpy=1.57079632679 0 1.57079632679, axis 0 1 0, limit lower=-2.8973 upper=2.8973 effort=87 velocity=2.1750
- added joint joint_ee: type fixed, parent link7, child end-effector, origin xyz=0 0 0.15 rpy=0 0 0
