Commit message: prepared experiments pose control

File: 00-experiment_pose_control/panda_arm_error.urdf (robot description, URDF)
Before this commit: robot panda, 8 links, 7 joints
Links:
- added link link8, mass 1.0
Joints:
- added joint joint8: type fixed, parent link7, child link8, origin xyz=0 0 0.107 rpy=0 0 0, axis 0 0 0
